File: Eagle/SDMAC.brd (EAGLE design)
At the start: 81.3 x 45.9 mm, 8 parts, among them IC1 SUPER_DMAC_THT, J1 CORTEX_DEBUG_PTH, U1 XC95288XL-10TQG144C, U2 NCP1117ST33T3G

Commit message: PCB Design Finished
Parts:
- removed C2: 10uF, Capacitor:CAPC2012X110
- removed J1: CORTEX_DEBUG_PTH, SparkFun-Connectors:2X5-PTH-1.27MM
- added A12: (no value), jumper:JP1
- added C10, C11, C12, C3, C4, C5, C6, C7, C8, C9: 0.1uF, Capacitor:CAPC2012X110
- added C13: 10uF, Volks73-Kemet:A
- added DMA, PWR, RD, WR: (no value), led:SML0805
- added R1, R2, R3, R4: 430, rcl:R0805
- added SV1: (no value), con-lstb:MA06-1
- moved U$1 20.9 mm to (49.4, 38.4)
- moved U$2 19.9 mm to (54.9, 25.9)
Connections:
- new net A12: A12.2, U1.15
- new net DMA_LED: DMA.C, U1.14
- new net N$1: PWR.A, R1.2
- new net N$2: R2.2, WR.A
- new net N$3: R3.2, RD.A
- new net N$4: DMA.A, R4.2
- new net RD_LED: RD.C, U1.13
- new net WR_LED: U1.12, WR.C
- net GND: now also A12.1, C10.2, C11.2, C12.2, C13.C, C3.2, C4.2, C5.2, C6.2, C7.2, C8.2, C9.2, PWR.C, SV1.5; no longer C2.2, J1.3, J1.5
- net TCK: now also SV1.4; no longer J1.4
- net TDI: now also SV1.2; no longer J1.8
- net TDO: now also SV1.3; no longer J1.6
- net TMS: now also SV1.1; no longer J1.2
- net VCC3.3: now also C10.1, C11.1, C12.1, C13.A, C3.1, C4.1, C5.1, C6.1, C7.1, C8.1, C9.1, R1.1, R2.1, R3.1, R4.1, SV1.6; no longer C2.1, J1.1
Routing:
- net VCC3.3: track 28.8 -> 77.3 mm
- net A12: track 0.00 -> 22.9 mm
- net TMS: track 23.7 -> 44.8 mm
- net WR_LED: track 0.00 -> 14.6 mm
- net N$3: track 0.00 -> 10.8 mm, vias 0 -> 1
- net RD_LED: track 0.00 -> 7.93 mm
- net DMA_LED: track 0.00 -> 6.49 mm
- net N$2: track 0.00 -> 6.31 mm, vias 0 -> 1
- net N$4: track 0.00 -> 6.11 mm, vias 0 -> 1
- net N$1: track 0.00 -> 3.99 mm, vias 0 -> 1
- net TDI: track 20.7 -> 22.8 mm
- net TCK: track 23.8 -> 24.8 mm
- net !IOW: track 19.3 -> 18.5 mm
- net !IOR: track 21.5 -> 20.9 mm
- net !DACK: track 18.1 -> 17.4 mm
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Other:
- board text added: "3.3V"
- board text added: "Design by M.Taylor 2022"
- board text added: "GND"
- board text added: "RE-SDMAC Prototype V0.1"
- board text added: "TCK"
- board text added: "TDI"
- board text added: "TDO"
- board text added: "TMS"
- board text added: "https://github.com/mbtaylor1982/SDMAC-Replacement"

Commit message: updated makefile, schmatics, gerbers etc...
Parts:
- added 5V: (no value), jumper:JP1
Connections:
- net !AS: now also U1.32; no longer U1.130
- net !CS: now also U1.3; no longer U1.121
- net !DS: now also U1.38; no longer U1.129
- net !RST: now also U1.143; no longer U1.120
- net CLK: now also U1.30; no longer U1.124
- net CPU_DATAD23: now also U1.17; no longer U1.3
- net CPU_DATAD24: now also U1.16; no longer U1.2
- net CPU_DATAD25: now also U1.142; no longer U1.143
- net GND: now also 5V.1
- net R!W: now also U1.2; no longer U1.131
- net VCC5: now also 5V.2
Routing:
- net !DS: track 56.7 -> 81.0 mm, vias 0 -> 2
- net CLK: track 50.1 -> 74.0 mm, vias 0 -> 4
- net !AS: track 61.8 -> 84.1 mm, vias 0 -> 2
- net !CS: track 44.2 -> 63.1 mm, vias 0 -> 4
- net !RST: track 45.1 -> 56.3 mm, vias 0 -> 2
- net R!W: track 60.9 -> 69.6 mm, vias 0 -> 2
- net CPU_DATAD24: track 91.5 -> 98.9 mm, vias 1 -> 3
- net CPU_DATAD23: track 66.7 -> 69.8 mm
- net VCC5: track 31.8 -> 34.2 mm
- net TDO: track 27.5 -> 29.2 mm
- net CPU_DATAD29: track 61.6 -> 62.3 mm
- net CPU_DATAD27: track 62.3 -> 62.9 mm
Other:
- board text added: "RE-SDMAC Prototype Rev A"
- board text removed: "RE-SDMAC Prototype V0.1"
