File: RE-SDMAC Rev B/SDMAC_revb.brd (EAGLE design)
At the start: 100 x 80 mm, 31 parts, among them IC1 SUPER_DMAC_THT, IC2 SN74LVCR162245A, IC3 SN74LVCR162245A, U1 SN74LVCH245APWPW20-M, U2 NCP1117ST33T3G

Commit message: More work on Rev B Prototype
Parts:
- removed 5V, A12: (no value), jumper:JP1
- removed C1: 10uF, Capacitor:CAPC2012X110
- removed C13: 10uF, Volks73-Kemet:A
- removed C3, C4, C5, C6, C7, C8: 0.1uF, Capacitor:CAPC2012X110
- removed DMA, PWR, RD, WR: (no value), led:SML0805
- removed IC2, IC3: SN74LVCR162245A, texas:DL_R-PDSO-G48
- removed R1, R2, R3, R4: 430, rcl:R0805
- removed U2: NCP1117ST33T3G, IC:SOT-223
- added U3, U4, U5: 74ALVC164245DGGRE4DGG48-M, 74alvc164254:DGG48-M
- U1: value SN74LVCH245APWPW20-M -> 74ALVC164245DGGRE4DGG48-M; device TI74LVC245:PW20-M -> 74alvc164254:DGG48-M
- moved C11 90.3 mm to (39.4, 45.7)
- moved C10 77.3 mm to (39.4, 66.0)
- moved C12 76.9 mm to (17.8, 45.7)
- moved U1 62.7 mm to (39.4, 58.4), turned to 0 degrees
- moved C9 50.7 mm to (17.8, 66.0)
- moved IC1 1.27 mm to (80.0, 47.0), turned to 180 degrees
Connections:
- removed net A12: A12.2
- removed net DMA_LED: DMA.C
- removed net N$1: PWR.A, R1.2
- removed net N$2: R2.2, WR.A
- removed net N$3: R3.2, RD.A
- removed net N$4: DMA.A, R4.2
- removed net RD_LED: RD.C
- removed net VCC: IC2.31, IC2.42, IC3.31, IC3.42, U1.20
- removed net WR_LED: WR.C
- new net !DATAOE: U1.25, U1.48, U3.25, U3.48
- new net P1-1: U4.30
- net !BERR: now also U5.11
- net !BG: now also U5.12
- net !BR: now also U4.13
- net !CS: now also U5.13
- net !CSS: now also U4.14, U4.48; no longer U1.19
- net !DACK: now also U4.16
- net !DMAEN: now also U4.17
- net !DREQ: now also U5.14
- net !INT2: now also U4.19
- net !IOR: now also U4.20
- net !IOW: now also U4.1, U4.22
- net !RST: now also U5.16
- net !STERM: now also U5.17
- net CLK: now also U5.23
- net CPU_ADDR2: now also U5.2
- net CPU_ADDR3: now also U5.3
- net CPU_ADDR4: now also U5.5
- net CPU_ADDR5: now also U5.6
- net CPU_ADDR6: now also U5.8
- net CPU_DATAD0: now also U1.2; no longer IC2.2
- net CPU_DATAD1: now also U1.3; no longer IC2.3
- net CPU_DATAD10: now also U1.16; no longer IC2.16
- net CPU_DATAD11: now also U1.17; no longer IC2.17
- net CPU_DATAD12: now also U1.19; no longer IC2.19
- net CPU_DATAD13: now also U1.20; no longer IC2.20
- net CPU_DATAD14: now also U1.22; no longer IC2.22
- net CPU_DATAD15: now also U1.23; no longer IC2.23
- net CPU_DATAD16: now also U3.2; no longer IC3.2
- net CPU_DATAD17: now also U3.3; no longer IC3.3
- net CPU_DATAD18: now also U3.5; no longer IC3.5
- net CPU_DATAD19: now also U3.6; no longer IC3.6
- net CPU_DATAD2: now also U1.5; no longer IC2.5
- net CPU_DATAD20: now also U3.8; no longer IC3.8
- net CPU_DATAD21: now also U3.9; no longer IC3.9
- net CPU_DATAD22: now also U3.11; no longer IC3.11
- net CPU_DATAD23: now also U3.12; no longer IC3.12
- net CPU_DATAD24: now also U3.13; no longer IC3.13
- net CPU_DATAD25: now also U3.14; no longer IC3.14
- net CPU_DATAD26: now also U3.16; no longer IC3.16
- net CPU_DATAD27: now also U3.17; no longer IC3.17
- net CPU_DATAD28: now also U3.19; no longer IC3.19
- net CPU_DATAD29: now also U3.20; no longer IC3.20
- net CPU_DATAD3: now also U1.6; no longer IC2.6
- net CPU_DATAD30: now also U3.22; no longer IC3.22
- net CPU_DATAD31: now also U3.23; no longer IC3.23
- net CPU_DATAD4: now also U1.8; no longer IC2.8
- net CPU_DATAD5: now also U1.9; no longer IC2.9
- net CPU_DATAD6: now also U1.11; no longer IC2.11
- net CPU_DATAD7: now also U1.12; no longer IC2.12
- net CPU_DATAD8: now also U1.13; no longer IC2.13
- net CPU_DATAD9: now also U1.14; no longer IC2.14
- net GND: now also U1.15, U1.21, U1.28, U1.34, U1.39, U1.4, U1.45, U3.10, U3.15, U3.21, U3.28, U3.34, U3.39, U3.4, U3.45, U4.10, U4.15, U4.21, U4.25, U4.28, U4.34, U4.39, U4.4, U4.45, U5.1, U5.10, U5.15, U5.19, U5.20, U5.21, U5.22, U5.24, U5.25, U5.28, U5.34, U5.39, U5.4, U5.45, U5.48; no longer 5V.1, A12.1, C1.2, C13.C, C3.2, C4.2, C5.2, C6.2, C7.2, C8.2, IC2.10, IC2.15, IC2.18, IC2.21, IC2.28, IC2.34, IC2.4, IC2.45, IC3.10, IC3.15, IC3.21, IC3.28, IC3.34, IC3.4, IC3.45, PWR.C, U2.1
- net INTA: now also U5.9
- net P_DATA0: now also U4.2; no longer U1.18
- net P_DATA1: now also U4.3; no longer U1.17
- net P_DATA2: now also U4.5; no longer U1.16
- net P_DATA3: now also U4.6; no longer U1.15
- net P_DATA4: now also U4.8; no longer U1.14
- net P_DATA5: now also U4.9; no longer U1.13
- net P_DATA6: now also U4.11; no longer U1.12
- net P_DATA7: now also U4.12; no longer U1.11
- net R!W: now also U1.1, U1.24, U3.1, U3.24; no longer IC2.1, IC2.24, IC3.1, IC3.24
- net SIZ1: now also U4.23
- net VCC3.3: now also U1.31, U1.42, U3.31, U3.42, U4.24, U4.31, U4.42, U5.31, U5.42; no longer C13.A, C3.1, C4.1, C5.1, C6.1, C7.1, C8.1, IC2.7, IC3.18, IC3.7, R1.1, R2.1, R3.1, R4.1, U2.2, U2.4
- net VCC5: now also U1.18, U1.7, U3.18, U3.7, U4.18, U4.7, U5.18, U5.7; no longer 5V.2, C1.1, U2.3

Commit message: more updates
Parts:
- added JP1: (no value), pinhead:1X02
- moved U5 34.1 mm to (41.9, 34.3), turned to 270 degrees
- moved U4 30.7 mm to (41.9, 57.1), turned to 270 degrees
- moved U1 29.2 mm to (22.9, 34.3), turned to 270 degrees
- moved U3 25.2 mm to (22.9, 57.1), turned to 270 degrees
- moved C11 12.6 mm to (33.8, 34.4), turned to 90 degrees
- moved C12 11.7 mm to (14.6, 34.4), turned to 90 degrees
- moved C10 10.3 mm to (33.8, 57.4), turned to 90 degrees
- moved C9 9.16 mm to (14.7, 57.4), turned to 90 degrees
- moved P1 4.58 mm to (30.5, 68.6)
- moved P2 3.59 mm to (7.62, 45.7)
- moved P3 2.84 mm to (30.5, 22.9)
- moved P4 1.80 mm to (53.3, 45.7), turned to 90 degrees
Connections:
- removed net P1-1: U4.30
- new net P1_HDR1: P1.1, U4.30
- new net P1_HDR10: P1.10, U5.43
- new net P1_HDR11: P1.11, U5.41
- new net P1_HDR12: P1.12, U4.48
- new net P1_HDR13: P1.13
- new net P1_HDR14: P1.14
- new net P1_HDR15: P1.15, U4.36
- new net P1_HDR16: P1.16, U4.33
- new net P1_HDR17: P1.17
- new net P1_HDR18: P1.18, U4.27
- new net P1_HDR19: P1.19
- new net P1_HDR2: P1.2, U4.32
- new net P1_HDR20: P1.20
- new net P1_HDR22: P1.22, U3.46
- new net P1_HDR23: P1.23, U3.37
- new net P1_HDR24: P1.24, U3.40
- new net P1_HDR3: P1.3, U4.29
- new net P1_HDR4: P1.4, U4.35
- new net P1_HDR5: P1.5, U1.27
- new net P1_HDR6: P1.6
- new net P1_HDR7: P1.7, U4.44
- new net P1_HDR8: P1.8, U5.32
- new net P1_HDR9: P1.9, U4.38
- new net P2_HDR10: P2.10, U3.35
- new net P2_HDR11: P2.11, U3.32
- new net P2_HDR12: P2.12, U5.37
- new net P2_HDR13: P2.13, U5.35
- new net P2_HDR14: P2.14, U5.26
- new net P2_HDR15: P2.15
- new net P2_HDR16: P2.16, U3.41
- new net P2_HDR17: P2.17, U3.38
- new net P2_HDR18: P2.18, U3.36
- new net P2_HDR19: P2.19, U3.33
- new net P2_HDR20: P2.20, U3.30
- new net P2_HDR21: P2.21, U4.46
- new net P2_HDR22: P2.22, U3.29
- new net P2_HDR23: P2.23, U3.27
- new net P2_HDR24: P2.24, U3.26
- new net P2_HDR25: P2.25
- new net P2_HDR26: P2.26
- new net P2_HDR3: P2.3
- new net P2_HDR4: P2.4, U3.44
- new net P2_HDR5: P2.5, U3.43
- new net P2_HDR6: P2.6
- new net P2_HDR7: P2.7, U4.47
- new net P2_HDR8: P2.8
- new net P2_HDR9: P2.9
- new net P3_HDR10: P3.10, U1.38
- new net P3_HDR11: P3.11, U1.36
- new net P3_HDR12: P3.12, U1.33
- new net P3_HDR13: P3.13, U1.30
- new net P3_HDR14: P3.14
- new net P3_HDR15: P3.15, U3.47
- new net P3_HDR16: P3.16
- new net P3_HDR17: P3.17
- new net P3_HDR18: P3.18, U1.46
- new net P3_HDR19: P3.19, U1.43
- new net P3_HDR20: P3.20, U1.40
- new net P3_HDR21: P3.21, U1.37
- new net P3_HDR22: P3.22, U1.35
- new net P3_HDR23: P3.23, U1.32
- new net P3_HDR24: P3.24, U1.29
- new net P3_HDR25: P3.25
- new net P3_HDR3: P3.3, U4.26
- new net P3_HDR4: P3.4
- new net P3_HDR5: P3.5
- new net P3_HDR6: P3.6, U1.47
- new net P3_HDR7: P3.7, U1.44
- new net P3_HDR8: P3.8, U1.41
- new net P3_HDR9: P3.9, U1.26
- new net P4_HDR11: P4.11, U5.36
- new net P4_HDR12: P4.12
- new net P4_HDR13: P4.13, U5.46
- new net P4_HDR14: P4.14, U5.47
- new net P4_HDR15: P4.15, U4.37
- new net P4_HDR16: P4.16, U4.40
- new net P4_HDR17: P4.17
- new net P4_HDR18: P4.18
- new net P4_HDR21: P4.21, U5.44
- new net P4_HDR22: P4.22, U5.33
- new net P4_HDR23: P4.23, U5.38
- new net P4_HDR24: P4.24, U5.40
- new net P4_HDR3: P4.3
- new net P4_HDR4: P4.4, U4.43
- new net P4_HDR5: P4.5
- new net P4_HDR6: P4.6, U4.41
- new net P4_HDR7: P4.7
- net !CSS: no longer U4.48
- net !DATAOE: now also P1.21
- net GND: now also JP1.2, P1.25, P1.26, P2.1, P2.2, P2.27, P3.1, P3.2, P3.26, P3.27, P4.1, P4.10, P4.2, P4.25, P4.26, P4.8, P4.9, U5.27, U5.29, U5.30
- net VCC3.3: now also P1.27, P1.28, P2.28, P3.28, P4.27, P4.28
- net VCC5: now also JP1.1
Routing:
- net VCC5: track 0.00 -> 134.6 mm
- net VCC3.3: track 0.00 -> 127.0 mm
- added copper zone on layer 1, net GND
- added copper zone on layer 16, net GND
Other:
- board size 100 x 80 mm -> 102.5 x 64.8 mm
