File: RE-SDMAC Rev B/SDMAC_revb.sch (EAGLE design)
At the start: 13 parts, among them IC1 SUPER_DMAC_THT, U1 74ALVC164245DGGRE4DGG48-M, U3 74ALVC164245DGGRE4DGG48-M, U4 74ALVC164245DGGRE4DGG48-M, U5 74ALVC164245DGGRE4DGG48-M

Commit message: quatus and rev b update
Parts:
- added JP1: (no value), pinhead:PINHD-1X2
Connections:
- removed net P1-1: U4A.2A5
- new net P1_HDR1: P1.1, U4A.2A5
- new net P1_HDR10: P1.10, U5A.1A4
- new net P1_HDR11: P1.11, U5A.1A5
- new net P1_HDR12: P1.12, U4A.!1OE
- new net P1_HDR13: P1.13
- new net P1_HDR14: P1.14
- new net P1_HDR15: P1.15, U4A.2A1
- new net P1_HDR16: P1.16, U4A.2A3
- new net P1_HDR17: P1.17
- new net P1_HDR18: P1.18, U4A.2A7
- new net P1_HDR19: P1.19
- new net P1_HDR2: P1.2, U4A.2A4
- new net P1_HDR20: P1.20
- new net P1_HDR22: P1.22, U3A.1A2
- new net P1_HDR23: P1.23, U3A.1A8
- new net P1_HDR24: P1.24, U3A.1A6
- new net P1_HDR3: P1.3, U4A.2A6
- new net P1_HDR4: P1.4, U4A.2A2
- new net P1_HDR5: P1.5, U1A.2A7
- new net P1_HDR6: P1.6
- new net P1_HDR7: P1.7, U4A.1A3
- new net P1_HDR8: P1.8, U5A.2A4
- new net P1_HDR9: P1.9, U4A.1A7
- new net P2_HDR10: P2.10, U3A.2A2
- new net P2_HDR11: P2.11, U3A.2A4
- new net P2_HDR12: P2.12, U5A.1A8
- new net P2_HDR13: P2.13, U5A.2A2
- new net P2_HDR14: P2.14, U5A.2A8
- new net P2_HDR15: P2.15
- new net P2_HDR16: P2.16, U3A.1A5
- new net P2_HDR17: P2.17, U3A.1A7
- new net P2_HDR18: P2.18, U3A.2A1
- new net P2_HDR19: P2.19, U3A.2A3
- new net P2_HDR20: P2.20, U3A.2A5
- new net P2_HDR21: P2.21, U4A.1A2
- new net P2_HDR22: P2.22, U3A.2A6
- new net P2_HDR23: P2.23, U3A.2A7
- new net P2_HDR24: P2.24, U3A.2A8
- new net P2_HDR25: P2.25
- new net P2_HDR26: P2.26
- new net P2_HDR3: P2.3
- new net P2_HDR4: P2.4, U3A.1A3
- new net P2_HDR5: P2.5, U3A.1A4
- new net P2_HDR6: P2.6
- new net P2_HDR7: P2.7, U4A.1A1
- new net P2_HDR8: P2.8
- new net P2_HDR9: P2.9
- new net P3_HDR10: P3.10, U1A.1A7
- new net P3_HDR11: P3.11, U1A.2A1
- new net P3_HDR12: P3.12, U1A.2A3
- new net P3_HDR13: P3.13, U1A.2A5
- new net P3_HDR14: P3.14
- new net P3_HDR15: P3.15, U3A.1A1
- new net P3_HDR16: P3.16
- new net P3_HDR17: P3.17
- new net P3_HDR18: P3.18, U1A.1A2
- new net P3_HDR19: P3.19, U1A.1A4
- new net P3_HDR20: P3.20, U1A.1A6
- new net P3_HDR21: P3.21, U1A.1A8
- new net P3_HDR22: P3.22, U1A.2A2
- new net P3_HDR23: P3.23, U1A.2A4
- new net P3_HDR24: P3.24, U1A.2A6
- new net P3_HDR25: P3.25
- new net P3_HDR3: P3.3, U4A.2A8
- new net P3_HDR4: P3.4
- new net P3_HDR5: P3.5
- new net P3_HDR6: P3.6, U1A.1A1
- new net P3_HDR7: P3.7, U1A.1A3
- new net P3_HDR8: P3.8, U1A.1A5
- new net P3_HDR9: P3.9, U1A.2A8
- new net P4_HDR11: P4.11, U5A.2A1
- new net P4_HDR12: P4.12
- new net P4_HDR13: P4.13, U5A.1A2
- new net P4_HDR14: P4.14, U5A.1A1
- new net P4_HDR15: P4.15, U4A.1A8
- new net P4_HDR16: P4.16, U4A.1A6
- new net P4_HDR17: P4.17
- new net P4_HDR18: P4.18
- new net P4_HDR21: P4.21, U5A.1A3
- new net P4_HDR22: P4.22, U5A.2A3
- new net P4_HDR23: P4.23, U5A.1A7
- new net P4_HDR24: P4.24, U5A.1A6
- new net P4_HDR3: P4.3
- new net P4_HDR4: P4.4, U4A.1A4
- new net P4_HDR5: P4.5
- new net P4_HDR6: P4.6, U4A.1A5
- new net P4_HDR7: P4.7
- net !CSS: no longer U4A.!1OE
- net !DATAOE: now also P1.21
- net GND: now also JP1.2, P1.25, P1.26, P2.1, P2.2, P2.27, P3.1, P3.2, P3.26, P3.27, P4.1, P4.10, P4.2, P4.25, P4.26, P4.8, P4.9, U5A.2A5, U5A.2A6, U5A.2A7
- net VCC3.3: now also P1.27, P1.28, P2.28, P3.28, P4.27, P4.28
- net VCC5: now also JP1.1
