File: RE-SDMAC Rev B/SDMAC_revb.sch (EAGLE design)
At the start: 31 parts, among them IC1 SUPER_DMAC_THT, IC2 SN74LVCR162245A, IC3 SN74LVCR162245A, U1 SN74LVCH245APWPW20-M, U2 NCP1117ST33T3G

Commit message: More work on Rev B Prototype
Parts:
- removed 5V, A12: (no value), jumper:JP1E
- removed C1: 10uF, Capacitor:C_CHIP-0805(2012-METRIC)
- removed C13: 10uF, Volks73-Kemet:T491A106K010AT
- removed C3, C4, C5, C6, C7, C8: 0.1uF, Capacitor:C_CHIP-0805(2012-METRIC)
- removed DMA, PWR, RD, WR: (no value), led:LEDSML0805
- removed IC2, IC3: SN74LVCR162245A, texas:SN74LVCR162245A
- removed R1, R2, R3, R4: 430, rcl:R-EU_R0805
- removed U2: NCP1117ST33T3G, IC:NCP1117ST33T3G
- added U3, U4, U5: 74ALVC164245DGGRE4DGG48-M, 74alvc164254:74ALVC164245DGGRE4DGG48-M
- U1: value SN74LVCH245APWPW20-M -> 74ALVC164245DGGRE4DGG48-M; device TI74LVC245:SN74LVCH245APWPW20-M -> 74alvc164254:74ALVC164245DGGRE4DGG48-M
Connections:
- removed net A12: A12.2
- removed net DMA_LED: DMA.C
- removed net N$1: PWR.A, R1.2
- removed net N$2: R2.2, WR.A
- removed net N$3: R3.2, RD.A
- removed net N$4: DMA.A, R4.2
- removed net RD_LED: RD.C
- removed net WR_LED: WR.C
- new net !DATAOE: U1A.!1OE, U1A.!2OE, U3A.!1OE, U3A.!2OE
- new net P1-1: U4A.2A5
- net !BERR: now also U5A.1B7
- net !BG: now also U5A.1B8
- net !BR: now also U4A.2B1
- net !CS: now also U5A.2B1
- net !CSS: now also U4A.!1OE, U4A.2B2; no longer U1.!OE
- net !DACK: now also U4A.2B3
- net !DMAEN: now also U4A.2B4
- net !DREQ: now also U5A.2B2
- net !INT2: now also U4A.2B5
- net !IOR: now also U4A.2B6
- net !IOW: now also U4A.1DIR, U4A.2B7
- net !RST: now also U5A.2B3
- net !STERM: now also U5A.2B4
- net CLK: now also U5A.2B8
- net CPU_ADDR2: now also U5A.1B1
- net CPU_ADDR3: now also U5A.1B2
- net CPU_ADDR4: now also U5A.1B3
- net CPU_ADDR5: now also U5A.1B4
- net CPU_ADDR6: now also U5A.1B5
- net CPU_DATAD0: now also U1A.1B1; no longer IC2.1B1
- net CPU_DATAD1: now also U1A.1B2; no longer IC2.1B2
- net CPU_DATAD10: now also U1A.2B3; no longer IC2.2B3
- net CPU_DATAD11: now also U1A.2B4; no longer IC2.2B4
- net CPU_DATAD12: now also U1A.2B5; no longer IC2.2B5
- net CPU_DATAD13: now also U1A.2B6; no longer IC2.2B6
- net CPU_DATAD14: now also U1A.2B7; no longer IC2.2B7
- net CPU_DATAD15: now also U1A.2B8; no longer IC2.2B8
- net CPU_DATAD16: now also U3A.1B1; no longer IC3.1B1
- net CPU_DATAD17: now also U3A.1B2; no longer IC3.1B2
- net CPU_DATAD18: now also U3A.1B3; no longer IC3.1B3
- net CPU_DATAD19: now also U3A.1B4; no longer IC3.1B4
- net CPU_DATAD2: now also U1A.1B3; no longer IC2.1B3
- net CPU_DATAD20: now also U3A.1B5; no longer IC3.1B5
- net CPU_DATAD21: now also U3A.1B6; no longer IC3.1B6
- net CPU_DATAD22: now also U3A.1B7; no longer IC3.1B7
- net CPU_DATAD23: now also U3A.1B8; no longer IC3.1B8
- net CPU_DATAD24: now also U3A.2B1; no longer IC3.2B1
- net CPU_DATAD25: now also U3A.2B2; no longer IC3.2B2
- net CPU_DATAD26: now also U3A.2B3; no longer IC3.2B3
- net CPU_DATAD27: now also U3A.2B4; no longer IC3.2B4
- net CPU_DATAD28: now also U3A.2B5; no longer IC3.2B5
- net CPU_DATAD29: now also U3A.2B6; no longer IC3.2B6
- net CPU_DATAD3: now also U1A.1B4; no longer IC2.1B4
- net CPU_DATAD30: now also U3A.2B7; no longer IC3.2B7
- net CPU_DATAD31: now also U3A.2B8; no longer IC3.2B8
- net CPU_DATAD4: now also U1A.1B5; no longer IC2.1B5
- net CPU_DATAD5: now also U1A.1B6; no longer IC2.1B6
- net CPU_DATAD6: now also U1A.1B7; no longer IC2.1B7
- net CPU_DATAD7: now also U1A.1B8; no longer IC2.1B8
- net CPU_DATAD8: now also U1A.2B1; no longer IC2.2B1
- net CPU_DATAD9: now also U1A.2B2; no longer IC2.2B2
- net GND: now also U1B.GND, U1B.GND_2, U1B.GND_3, U1B.GND_4, U1B.GND_5, U1B.GND_6, U1B.GND_7, U1B.GND_8, U3B.GND, U3B.GND_2, U3B.GND_3, U3B.GND_4, U3B.GND_5, U3B.GND_6, U3B.GND_7, U3B.GND_8, U4A.!2OE, U4B.GND, U4B.GND_2, U4B.GND_3, U4B.GND_4, U4B.GND_5, U4B.GND_6, U4B.GND_7, U4B.GND_8, U5A.!1OE, U5A.!2OE, U5A.1DIR, U5A.2B5, U5A.2B6, U5A.2B7, U5A.2DIR, U5B.GND, U5B.GND_2, U5B.GND_3, U5B.GND_4, U5B.GND_5, U5B.GND_6, U5B.GND_7, U5B.GND_8; no longer 5V.1, A12.1, C1.2, C13.C, C3.2, C4.2, C5.2, C6.2, C7.2, C8.2, IC2.GND, IC2.GND@1, IC2.GND@2, IC2.GND@3, IC2.VCC@1, IC3.GND, IC3.GND@1, IC3.GND@2, IC3.GND@3, PWR.C, U2.ADJ/GND
- net INTA: now also U5A.1B6
- net P_DATA0: now also U4A.1B1; no longer U1.B1
- net P_DATA1: now also U4A.1B2; no longer U1.B2
- net P_DATA2: now also U4A.1B3; no longer U1.B3
- net P_DATA3: now also U4A.1B4; no longer U1.B4
- net P_DATA4: now also U4A.1B5; no longer U1.B5
- net P_DATA5: now also U4A.1B6; no longer U1.B6
- net P_DATA6: now also U4A.1B7; no longer U1.B7
- net P_DATA7: now also U4A.1B8; no longer U1.B8
- net R!W: now also U1A.1DIR, U1A.2DIR, U3A.1DIR, U3A.2DIR; no longer IC2.1DIR, IC2.2DIR, IC3.1DIR, IC3.2DIR
- net SIZ1: now also U4A.2B8
- net VCC3.3: now also U1B.VCCA, U1B.VCCA_2, U3B.VCCA, U3B.VCCA_2, U4A.2DIR, U4B.VCCA, U4B.VCCA_2, U5B.VCCA, U5B.VCCA_2; no longer C13.A, C3.1, C4.1, C5.1, C6.1, C7.1, C8.1, IC2.VCC, IC3.VCC, IC3.VCC@1, R1.1, R2.1, R3.1, R4.1, U2.4, U2.OUT
- net VCC5: now also U1B.VCCB, U1B.VCCB_2, U3B.VCCB, U3B.VCCB_2, U4B.VCCB, U4B.VCCB_2, U5B.VCCB, U5B.VCCB_2; no longer 5V.2, C1.1, U2.IN
Other:
- moved on the sheet: P1, P2, P3, P4

Commit message: more updates
Parts:
- added JP1: (no value), pinhead:PINHD-1X2
Connections:
- removed net P1-1: U4A.2A5
- new net P1_HDR1: P1.1, U4A.2A5
- new net P1_HDR10: P1.10, U5A.1A4
- new net P1_HDR11: P1.11, U5A.1A5
- new net P1_HDR12: P1.12, U4A.!1OE
- new net P1_HDR13: P1.13
- new net P1_HDR14: P1.14
- new net P1_HDR15: P1.15, U4A.2A1
- new net P1_HDR16: P1.16, U4A.2A3
- new net P1_HDR17: P1.17
- new net P1_HDR18: P1.18, U4A.2A7
- new net P1_HDR19: P1.19
- new net P1_HDR2: P1.2, U4A.2A4
- new net P1_HDR20: P1.20
- new net P1_HDR22: P1.22, U3A.1A2
- new net P1_HDR23: P1.23, U3A.1A8
- new net P1_HDR24: P1.24, U3A.1A6
- new net P1_HDR3: P1.3, U4A.2A6
- new net P1_HDR4: P1.4, U4A.2A2
- new net P1_HDR5: P1.5, U1A.2A7
- new net P1_HDR6: P1.6
- new net P1_HDR7: P1.7, U4A.1A3
- new net P1_HDR8: P1.8, U5A.2A4
- new net P1_HDR9: P1.9, U4A.1A7
- new net P2_HDR10: P2.10, U3A.2A2
- new net P2_HDR11: P2.11, U3A.2A4
- new net P2_HDR12: P2.12, U5A.1A8
- new net P2_HDR13: P2.13, U5A.2A2
- new net P2_HDR14: P2.14, U5A.2A8
- new net P2_HDR15: P2.15
- new net P2_HDR16: P2.16, U3A.1A5
- new net P2_HDR17: P2.17, U3A.1A7
- new net P2_HDR18: P2.18, U3A.2A1
- new net P2_HDR19: P2.19, U3A.2A3
- new net P2_HDR20: P2.20, U3A.2A5
- new net P2_HDR21: P2.21, U4A.1A2
- new net P2_HDR22: P2.22, U3A.2A6
- new net P2_HDR23: P2.23, U3A.2A7
- new net P2_HDR24: P2.24, U3A.2A8
- new net P2_HDR25: P2.25
- new net P2_HDR26: P2.26
- new net P2_HDR3: P2.3
- new net P2_HDR4: P2.4, U3A.1A3
- new net P2_HDR5: P2.5, U3A.1A4
- new net P2_HDR6: P2.6
- new net P2_HDR7: P2.7, U4A.1A1
- new net P2_HDR8: P2.8
- new net P2_HDR9: P2.9
- new net P3_HDR10: P3.10, U1A.1A7
- new net P3_HDR11: P3.11, U1A.2A1
- new net P3_HDR12: P3.12, U1A.2A3
- new net P3_HDR13: P3.13, U1A.2A5
- new net P3_HDR14: P3.14
- new net P3_HDR15: P3.15, U3A.1A1
- new net P3_HDR16: P3.16
- new net P3_HDR17: P3.17
- new net P3_HDR18: P3.18, U1A.1A2
- new net P3_HDR19: P3.19, U1A.1A4
- new net P3_HDR20: P3.20, U1A.1A6
- new net P3_HDR21: P3.21, U1A.1A8
- new net P3_HDR22: P3.22, U1A.2A2
- new net P3_HDR23: P3.23, U1A.2A4
- new net P3_HDR24: P3.24, U1A.2A6
- new net P3_HDR25: P3.25
- new net P3_HDR3: P3.3, U4A.2A8
- new net P3_HDR4: P3.4
- new net P3_HDR5: P3.5
- new net P3_HDR6: P3.6, U1A.1A1
- new net P3_HDR7: P3.7, U1A.1A3
- new net P3_HDR8: P3.8, U1A.1A5
- new net P3_HDR9: P3.9, U1A.2A8
- new net P4_HDR11: P4.11, U5A.2A1
- new net P4_HDR12: P4.12
- new net P4_HDR13: P4.13, U5A.1A2
- new net P4_HDR14: P4.14, U5A.1A1
- new net P4_HDR15: P4.15, U4A.1A8
- new net P4_HDR16: P4.16, U4A.1A6
- new net P4_HDR17: P4.17
- new net P4_HDR18: P4.18
- new net P4_HDR21: P4.21, U5A.1A3
- new net P4_HDR22: P4.22, U5A.2A3
- new net P4_HDR23: P4.23, U5A.1A7
- new net P4_HDR24: P4.24, U5A.1A6
- new net P4_HDR3: P4.3
- new net P4_HDR4: P4.4, U4A.1A4
- new net P4_HDR5: P4.5
- new net P4_HDR6: P4.6, U4A.1A5
- new net P4_HDR7: P4.7
- net !CSS: no longer U4A.!1OE
- net !DATAOE: now also P1.21
- net GND: now also JP1.2, P1.25, P1.26, P2.1, P2.2, P2.27, P3.1, P3.2, P3.26, P3.27, P4.1, P4.10, P4.2, P4.25, P4.26, P4.8, P4.9, U5A.2A5, U5A.2A6, U5A.2A7
- net VCC3.3: now also P1.27, P1.28, P2.28, P3.28, P4.27, P4.28
- net VCC5: now also JP1.1
